Commit message: add hardware and bringup for arm

File: ros2_control_demo_description/rrdiffbot_description/ros2_control/arm.ros2_control.urdf.xacro (robot description, xacro)
@@ -4,13 +4,13 @@
     <ros2_control name="${name}" type="system">
       <hardware>
-        <plugin>ros2_control_demo_hardware/ArmSystemPositionOnlyHardware</plugin>
+        <plugin>ros2_control_demo_hardware/rrdiffbot/RRDiffBotArmSystemPositionOnlyHardware</plugin>
         <param name="example_param_hw_start_duration_sec">0</param>
         <param name="example_param_hw_stop_duration_sec">3.0</param>
-        <param name="example_param_hw_slowdown">100</param>
+        <param name="example_param_hw_slowdown">10</param>
       </hardware>
       <joint name="${prefix}joint1">
         <command_interface name="position">
-          <param name="min">-1</param>
-          <param name="max">1</param>
+          <param name="min">${-pi/2}</param>
+          <param name="max">${pi/2}</param>
         </command_interface>
         <state_interface name="position"/>
@@ -18,6 +18,6 @@
       <joint name="${prefix}joint2">
         <command_interface name="position">
-          <param name="min">-1</param>
-          <param name="max">1</param>
+          <param name="min">${-pi/2}</param>
+          <param name="max">${pi/2}</param>
         </command_interface>
         <state_interface name="position"/>

File: ros2_control_demo_description/rrdiffbot_description/urdf/arm_description.urdf.xacro (robot description, xacro)
@@ -6,5 +6,5 @@
   <xacro:property name="width" value="0.075" /> <!-- Square dimensions (widthxwidth) of beams -->
   <xacro:property name="height1" value="0.5" /> <!-- Link 1 -->
-  <xacro:property name="height2" value="0.5" /> <!-- Link 2 -->
+  <xacro:property name="height2" value="0.28" /> <!-- Link 2 -->
   <xacro:property name="height3" value="0.5" /> <!-- Link 3 -->
   <xacro:property name="axel_offset" value="0.05" /> <!-- Space btw top of beam and the each joint -->
@@ -108,10 +108,4 @@
         <link name="${prefix}tool_link">
         </link>
-        <joint name="${prefix}hokuyo_joint" type="fixed">
-          <axis xyz="0 1 0" />
-          <origin xyz="0 0 ${height3 - axel_offset/2}" rpy="0 0 0"/>
-          <parent link="${prefix}link2"/>
-          <child link="${prefix}hokuyo_link"/>
-        </joint>
   </xacro:macro>
 </robot>
