Commit message: base changes for two subsystems

File: ros2_control_demo_description/rrbot_description/urdf/rrbot_description.urdf.xacro (robot description, xacro)
@@ -1,5 +1,5 @@
 <?xml version="1.0"?>
 <robot xmlns:xacro="http://www.ros.org/wiki/xacro">
-  <xacro:macro name="rrbot" params="parent prefix *origin">
+  <xacro:macro name="rrbot" params="parent prefix base_color *origin">
   <!-- Constants for robot dimensions -->
   <xacro:property name="mass" value="1" /> <!-- arbitrary value for mass -->
@@ -28,5 +28,5 @@
         <box size="${width} ${width} ${height1}"/>
       </geometry>
-      <material name="orange"/>
+      <material name="${base_color}"/>
     </visual>
     <inertial>

File: ros2_control_demo_description/two_distributed_rrbots_description/ros2_control/rrbot_two.ros2_control.xacro (robot description, xacro)
@@ -1,5 +1,5 @@
 <?xml version="1.0"?>
 <robot xmlns:xacro="http://www.ros.org/wiki/xacro">
-  <xacro:macro name="rrbot_two" params="name prefix">
+  <xacro:macro name="rrbot_two_hw" params="name prefix">
     <ros2_control name="${name}" type="system">
       <hardware>

File: ros2_control_demo_description/two_distributed_rrbots_description/urdf/main.urdf.xacro (robot description, xacro)
@@ -5,5 +5,5 @@
 https://github.com/ros-simulation/gazebo_ros_demos/blob/kinetic-devel/rrbot_description/urdf/rrbot.xacro
 -->
-<robot xmlns:xacro="http://www.ros.org/wiki/xacro" name="rrbot_one">
+<robot xmlns:xacro="http://www.ros.org/wiki/xacro" name="2dof_robot">
   <xacro:arg name="prefix" default="" />
   <!-- Import RRBot macro -->
@@ -12,5 +12,5 @@
   <xacro:include filename="$(find rrbot_description)/gazebo/rrbot.materials.xacro" />
   <!-- Import RRBot ros2_control description -->
-  <xacro:include filename="$(find two_distributed_rrbots_description)/ros2_control/rrbot_one.ros2_control.xacro" />
+  <xacro:include filename="$(find rrbot_description)/ros2_control/rrbot.ros2_control.xacro" />
   <!-- Used for fixing robot -->
   <link name="world"/>
@@ -18,9 +18,8 @@
     <static>true</static>
   </gazebo>
-  <!-- First rrbot-->
-  <xacro:rrbot parent="world" prefix="$(arg prefix)">
-    <origin xyz="2 0 0" rpy="0 0 0" />
+  <xacro:rrbot parent="world" prefix="$(arg prefix)" base_color="red">
+    <origin xyz="0 3 0" rpy="0 0 0" />
   </xacro:rrbot>
-  <xacro:rrbot_one_hw
-    name="rrbot_satellite_1" prefix="$(arg prefix)" />
+  <xacro:rrbot_ros2_control
+    name="RRBot" prefix="$(arg prefix)" />
 </robot>

File: ros2_control_demo_description/two_distributed_rrbots_description/urdf/two_distributed_rrbots_one.urdf.xacro (robot description, xacro)
@@ -19,5 +19,5 @@
   </gazebo>
   <!-- First rrbot-->
-  <xacro:rrbot parent="world" prefix="$(arg prefix)">
+  <xacro:rrbot parent="world" prefix="$(arg prefix)" base_color="green">
     <origin xyz="2 0 0" rpy="0 0 0" />
   </xacro:rrbot>

File: ros2_control_demo_description/two_distributed_rrbots_description/urdf/two_distributed_rrbots_two.urdf.xacro (robot description, xacro)
@@ -5,5 +5,5 @@
 https://github.com/ros-simulation/gazebo_ros_demos/blob/kinetic-devel/rrbot_description/urdf/rrbot.xacro
 -->
-<robot xmlns:xacro="http://www.ros.org/wiki/xacro" name="2dof_robot">
+<robot xmlns:xacro="http://www.ros.org/wiki/xacro" name="rrbot_one">
   <xacro:arg name="prefix" default="" />
   <!-- Import RRBot macro -->
@@ -12,5 +12,5 @@
   <xacro:include filename="$(find rrbot_description)/gazebo/rrbot.materials.xacro" />
   <!-- Import RRBot ros2_control description -->
-  <xacro:include filename="$(find rrbot_description)/ros2_control/rrbot.ros2_control.xacro" />
+  <xacro:include filename="$(find two_distributed_rrbots_description)/ros2_control/rrbot_two.ros2_control.xacro" />
   <!-- Used for fixing robot -->
   <link name="world"/>
@@ -18,8 +18,9 @@
     <static>true</static>
   </gazebo>
-  <xacro:rrbot parent="world" prefix="$(arg prefix)" base_color="orange">
-    <origin xyz="0 0 0" rpy="0 0 0" />
+  <!-- second rrbot-->
+  <xacro:rrbot parent="world" prefix="$(arg prefix)" base_color="blue">
+    <origin xyz="-2 0 0" rpy="0 0 0" />
   </xacro:rrbot>
-  <xacro:rrbot_ros2_control
-    name="RRBot" prefix="$(arg prefix)" />
+  <xacro:rrbot_two_hw
+    name="rrbot_satellite_2" prefix="$(arg prefix)" />
 </robot>
