Commit message: add colors for base to distinguish robotis

File: ros2_control_demo_description/rrbot_description/urdf/rrbot.urdf.xacro (robot description, xacro)
@@ -18,5 +18,5 @@
     <static>true</static>
   </gazebo>
-  <xacro:rrbot parent="world" prefix="$(arg prefix)" base_color="orange">
+  <xacro:rrbot parent="world" prefix="$(arg prefix)">
     <origin xyz="0 0 0" rpy="0 0 0" />
   </xacro:rrbot>

File: ros2_control_demo_description/rrbot_description/urdf/rrbot_description.urdf.xacro (robot description, xacro)
@@ -1,5 +1,5 @@
 <?xml version="1.0"?>
 <robot xmlns:xacro="http://www.ros.org/wiki/xacro">
-  <xacro:macro name="rrbot" params="parent prefix base_color *origin">
+  <xacro:macro name="rrbot" params="parent prefix base_color='orange' *origin">
   <!-- Constants for robot dimensions -->
   <xacro:property name="mass" value="1" /> <!-- arbitrary value for mass -->

File: ros2_control_demo_description/two_distributed_rrbots_description/urdf/main.urdf.xacro (robot description, xacro)
@@ -7,4 +7,5 @@
 <robot xmlns:xacro="http://www.ros.org/wiki/xacro" name="2dof_robot">
   <xacro:arg name="prefix" default="" />
+  <xacro:arg name="base_color" default="orange" />
   <!-- Import RRBot macro -->
   <xacro:include filename="$(find rrbot_description)/urdf/rrbot_description.urdf.xacro" />
@@ -18,5 +19,5 @@
     <static>true</static>
   </gazebo>
-  <xacro:rrbot parent="world" prefix="$(arg prefix)" base_color="red">
+  <xacro:rrbot parent="world" prefix="$(arg prefix)" base_color="$(arg base_color)">
     <origin xyz="0 3 0" rpy="0 0 0" />
   </xacro:rrbot>

File: ros2_control_demo_description/two_distributed_rrbots_description/urdf/two_distributed_rrbots_one.urdf.xacro (robot description, xacro)
@@ -7,4 +7,5 @@
 <robot xmlns:xacro="http://www.ros.org/wiki/xacro" name="rrbot_one">
   <xacro:arg name="prefix" default="" />
+  <xacro:arg name="base_color" default="orange" />
   <!-- Import RRBot macro -->
   <xacro:include filename="$(find rrbot_description)/urdf/rrbot_description.urdf.xacro" />
@@ -19,5 +20,5 @@
   </gazebo>
   <!-- First rrbot-->
-  <xacro:rrbot parent="world" prefix="$(arg prefix)" base_color="green">
+  <xacro:rrbot parent="world" prefix="$(arg prefix)" base_color="$(arg base_color)">
     <origin xyz="2 0 0" rpy="0 0 0" />
   </xacro:rrbot>

File: ros2_control_demo_description/two_distributed_rrbots_description/urdf/two_distributed_rrbots_two.urdf.xacro (robot description, xacro)
@@ -7,4 +7,5 @@
 <robot xmlns:xacro="http://www.ros.org/wiki/xacro" name="rrbot_one">
   <xacro:arg name="prefix" default="" />
+  <xacro:arg name="base_color" default="orange" />
   <!-- Import RRBot macro -->
   <xacro:include filename="$(find rrbot_description)/urdf/rrbot_description.urdf.xacro" />
@@ -19,5 +20,5 @@
   </gazebo>
   <!-- second rrbot-->
-  <xacro:rrbot parent="world" prefix="$(arg prefix)" base_color="blue">
+  <xacro:rrbot parent="world" prefix="$(arg prefix)" base_color="$(arg base_color)">
     <origin xyz="-2 0 0" rpy="0 0 0" />
   </xacro:rrbot>
